File: hardware/kicad/ozsec2025/ozsec2025.kicad_sch (KiCad schematic)
At the start: 84 parts, among them J1 USB_C_Receptacle_USB2.0, J2 PIN_RPS, J4 SM03B-SRSS-TB, SW1 POWER, SW10 SW_A, SW11 SW_B, SW2 BOOT, SW3 RESET, SW4 SW_START, SW5 SW_UP, SW6 SW_DOWN, SW7 SW_LEFT, SW8 SW_RIGHT, SW9 SW_SELECT, U1 TLV1117LV-33, U2 RP2350_80QFN, U3 USBLC6-2SC6, U4 ME4054BM5G-N, U5 W25Q128JVS, Y1 ABM8-272-T3

Commit message: Update footprints
Parts:
- BT1: footprint ozsec:MY-AA-04 -> ozsec-common:MY-AA-04
- BT1A1: footprint ozsec:MY-AA-04_BT1A -> ozsec-common:MY-AA-04_BT1A
- BT1B1: footprint ozsec:MY-AA-04_BT1B -> ozsec-common:MY-AA-04_BT1B
- U2: footprint ozsec:RP2350-QFN-80-1EP_10x10_P0.4mm_EP3.4x3.4mm_ThermalVias -> ozsec-common:RP2350-QFN-80-1EP_10x10_P0.4mm_EP3.4x3.4mm_ThermalVias
Changed lines of the file:
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@@
 			)
 		)
-		(property "Footprint" "ozsec:MY-AA-04_BT1A"
+		(property "Footprint" "ozsec-common:MY-AA-04_BT1A"
 			(at -3.81 116.586 90)
 			(effects
@@
 			)
 		)
-		(property "Footprint" "ozsec:RP2350-QFN-80-1EP_10x10_P0.4mm_EP3.4x3.4mm_ThermalVias"
+		(property "Footprint" "ozsec-common:RP2350-QFN-80-1EP_10x10_P0.4mm_EP3.4x3.4mm_ThermalVias"
 			(at 149.86 107.95 0)
 			(effects
@@
 			)
 		)
-		(property "Footprint" "ozsec:MY-AA-04"
+		(property "Footprint" "ozsec-common:MY-AA-04"
 			(at 17.78 122.936 90)
 			(effects
@@
 			)
 		)
-		(property "Footprint" "ozsec:MY-AA-04_BT1B"
+		(property "Footprint" "ozsec-common:MY-AA-04_BT1B"
 			(at -3.81 128.016 90)
 			(effects
