File: hardware/kicad/ozsec2025/ozsec2025.kicad_pcb (KiCad board)
At the start: 2 copper layers, 88.6 x 92.6 mm, 65 parts, among them J1 USB_C_Receptacle_USB2.0, J2 PIN_RPS, J4 SM03B-SRSS-TB, SW1 POWER, SW10 SW_A, SW11 SW_B, SW2 BOOT, SW3 RESET, SW4 SW_START, SW5 SW_UP, SW6 SW_DOWN, SW7 SW_LEFT, SW8 SW_RIGHT, SW9 SW_SELECT, U1 TLV1117LV-33, U2 RP2350_80QFN, U3 USBLC6-2SC6, U4 ME4054BM5G-N, Y1 ABM8-272-T3

Commit message: Clean slate on PCB.
Parts:
- removed BT1: Battery, ozsec:MY-AA-04
- removed BT1A1: Battery Terminal, ozsec:MY-AA-04_BT1A
- removed BT1B1: Battery Terminal, ozsec:MY-AA-04_BT1B
- removed C10, C13, C14, C15, C16, C17, C18, C19, C20, C22, C23, C5: 100nF, Capacitor_SMD:C_0402_1005Metric
- removed C11, C12: 4.7uF, Capacitor_SMD:C_0402_1005Metric
- removed C2: 0.1uF, Capacitor_SMD:C_0402_1005Metric
- removed C21: 10u, Capacitor_SMD:C_0805_2012Metric
- removed C3: 100uF, Capacitor_SMD:C_1206_3216Metric
- removed C4: 1uF, Capacitor_SMD:C_0402_1005Metric
- removed C6, C7: 15p, Capacitor_SMD:C_0402_1005Metric
- removed D45: CHARGING, LED_SMD:LED_0805_2012Metric_Pad1.15x1.40mm_HandSolder
- removed D46: POWER, LED_SMD:LED_0805_2012Metric_Pad1.15x1.40mm_HandSolder
- removed F1: Fuse, Fuse:Fuse_1206_3216Metric
- removed J1: USB_C_Receptacle_USB2.0, Connector_USB:USB_C_Receptacle_G-Switch_GT-USB-7010ASV
- removed J2: PIN_RPS, Connector_PinHeader_2.54mm:PinHeader_1x02_P2.54mm_Horizontal
- removed J4: SM03B-SRSS-TB, Connector_JST:JST_SH_SM03B-SRSS-TB_1x03-1MP_P1.00mm_Horizontal
- removed R1, R2: 5.1K, Resistor_SMD:R_0402_1005Metric
- removed R10: 0, Resistor_SMD:R_0402_1005Metric
- removed R11: 33, Resistor_SMD:R_0402_1005Metric
- removed R12, R7, R8: 1k, Resistor_SMD:R_0402_1005Metric
- removed R13, R14: 27, Resistor_SMD:R_0402_1005Metric
- removed R3, R4: 2K, Resistor_SMD:R_0402_1005Metric
- removed R5: 1K, Resistor_SMD:R_0402_1005Metric
- removed R6, R9: DNF, Resistor_SMD:R_0402_1005Metric
- removed the REF** at (159.8, 92.5) (x2)
- removed the REF** at (114.5, 63.5)
- removed SW1: POWER, Button_Switch_SMD:SW_SPDT_PCM12
- removed SW10: SW_A, Button_Switch_SMD:SW_Push_1P1T_XKB_TS-1187A
- removed SW11: SW_B, Button_Switch_SMD:SW_Push_1P1T_XKB_TS-1187A
- removed SW2: BOOT, Button_Switch_SMD:SW_Push_1P1T_XKB_TS-1187A
- removed SW3: RESET, Button_Switch_SMD:SW_Push_1P1T_XKB_TS-1187A
- removed SW4: SW_START, Button_Switch_SMD:SW_Push_1P1T_XKB_TS-1187A
- removed SW5: SW_UP, Button_Switch_SMD:SW_Push_1P1T_XKB_TS-1187A
- removed SW6: SW_DOWN, Button_Switch_SMD:SW_Push_1P1T_XKB_TS-1187A
- removed SW7: SW_LEFT, Button_Switch_SMD:SW_Push_1P1T_XKB_TS-1187A
- removed SW8: SW_RIGHT, Button_Switch_SMD:SW_Push_1P1T_XKB_TS-1187A
- removed SW9: SW_SELECT, Button_Switch_SMD:SW_Push_1P1T_XKB_TS-1187A
- removed TP1: VBUS, TestPoint:TestPoint_Pad_D1.5mm
- removed TP2: +3.3V, TestPoint:TestPoint_Pad_D1.5mm
- removed TP3: GND, TestPoint:TestPoint_Pad_1.5x1.5mm
- removed U1: TLV1117LV-33, Package_TO_SOT_SMD:SOT-223
- removed U2: RP2350_80QFN, ozsec:RP2350-QFN-80-1EP_10x10_P0.4mm_EP3.4x3.4mm_ThermalVias
- removed U3: USBLC6-2SC6, Package_TO_SOT_SMD:SOT-23-6
- removed U4: ME4054BM5G-N, Package_TO_SOT_SMD:TSOT-23-5
- removed Y1: ABM8-272-T3, Crystal:Crystal_SMD_3225-4Pin_3.2x2.5mm
- added REF**: Floppy_Slide_Cu, ozsec-2025:Floppy_Slide_Cu, F.Cu at (147.0, 113.8)
- added REF**: Floppy_Outline_Edge, ozsec-2025:Floppy_Outline_Edge, F.Cu at (102.0, 84.2)
Routing:
- net GND: track 65.5 -> 0.00 mm, vias 10 -> 0
- net VBUS: track 35.7 -> 0.00 mm
- net unconnected-(BT1A1-+-Pad1): track 20.7 -> 0.00 mm, vias 1 -> 0
- net unconnected-(BT1B1---Pad2): track 13.1 -> 0.00 mm
- net +3V3: track 13.0 -> 0.00 mm
- net /USB_D+: track 10.5 -> 0.00 mm
- net /USB_D-: track 9.74 -> 0.00 mm
- net Net-(J1-CC1): track 6.94 -> 0.00 mm
- net Net-(J1-CC2): track 6.39 -> 0.00 mm
- net +3.3: track 6.30 -> 0.00 mm
- net /GPIO7: track 6.00 -> 0.00 mm
- net /GPIO6: track 6.00 -> 0.00 mm
- net /GPIO5: track 6.00 -> 0.00 mm
- net /GPIO4: track 6.00 -> 0.00 mm
- net /GPIO3: track 6.00 -> 0.00 mm
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Other:
- outline, holes or cut-outs redrawn
